Commit message: Correct robot name to r820

File: iiwa_14_r820_robot_description/urdf/iiwa_14_r820.urdf.xacro (robot description, xacro)
@@ -1,16 +1,16 @@
 <?xml version="1.0"?>
 <robot xmlns:xacro="http://ros.org/wiki/xacro">
-    <xacro:macro name="iiwa_14_r850" params="parent *origin prefix">
+    <xacro:macro name="iiwa_14_r820" params="parent *origin prefix">
         <link name="${prefix}base_link">
             <visual>
                 <origin xyz="0 0 0" rpy="0 0 0"/>
                 <geometry>
-                    <mesh filename="package://iiwa_14_r850_robot_description/meshes/base.dae" scale="1 1 1"/>
-                </geometry>
-            </visual>
-            <collision>
-                <origin xyz="0 0 0" rpy="0 0 0"/>
-                <geometry>
-                    <mesh filename="package://iiwa_14_r850_robot_description/meshes/base.dae" scale="1 1 1"/>
+                    <mesh filename="package://iiwa_14_r820_robot_description/meshes/base.dae" scale="1 1 1"/>
+                </geometry>
+            </visual>
+            <collision>
+                <origin xyz="0 0 0" rpy="0 0 0"/>
+                <geometry>
+                    <mesh filename="package://iiwa_14_r820_robot_description/meshes/base.dae" scale="1 1 1"/>
                 </geometry>
             </collision>
@@ -30,11 +30,11 @@
                 <origin xyz="0 0 0" rpy="0 0 0"/>
                 <geometry>
-                    <mesh filename="package://iiwa_14_r850_robot_description/meshes/link1.dae" scale="1 1 1"/>
-                </geometry>
-            </visual>
-            <collision>
-                <origin xyz="0 0 0" rpy="0 0 0"/>
-                <geometry>
-                    <mesh filename="package://iiwa_14_r850_robot_description/meshes/link1.dae" scale="1 1 1"/>
+                    <mesh filename="package://iiwa_14_r820_robot_description/meshes/link1.dae" scale="1 1 1"/>
+                </geometry>
+            </visual>
+            <collision>
+                <origin xyz="0 0 0" rpy="0 0 0"/>
+                <geometry>
+                    <mesh filename="package://iiwa_14_r820_robot_description/meshes/link1.dae" scale="1 1 1"/>
                 </geometry>
             </collision>
@@ -57,11 +57,11 @@
                 <origin xyz="0 0 0" rpy="0 0 0"/>
                 <geometry>
-                    <mesh filename="package://iiwa_14_r850_robot_description/meshes/link2.dae" scale="1 1 1"/>
-                </geometry>
-            </visual>
-            <collision>
-                <origin xyz="0 0 0" rpy="0 0 0"/>
-                <geometry>
-                    <mesh filename="package://iiwa_14_r850_robot_description/meshes/link2.dae" scale="1 1 1"/>
+                    <mesh filename="package://iiwa_14_r820_robot_description/meshes/link2.dae" scale="1 1 1"/>
+                </geometry>
+            </visual>
+            <collision>
+                <origin xyz="0 0 0" rpy="0 0 0"/>
+                <geometry>
+                    <mesh filename="package://iiwa_14_r820_robot_description/meshes/link2.dae" scale="1 1 1"/>
                 </geometry>
             </collision>
@@ -84,11 +84,11 @@
                 <origin xyz="0 0 0" rpy="0 0 0"/>
                 <geometry>
-                    <mesh filename="package://iiwa_14_r850_robot_description/meshes/link3.dae" scale="1 1 1"/>
-                </geometry>
-            </visual>
-            <collision>
-                <origin xyz="0 0 0" rpy="0 0 0"/>
-                <geometry>
-                    <mesh filename="package://iiwa_14_r850_robot_description/meshes/link3.dae" scale="1 1 1"/>
+                    <mesh filename="package://iiwa_14_r820_robot_description/meshes/link3.dae" scale="1 1 1"/>
+                </geometry>
+            </visual>
+            <collision>
+                <origin xyz="0 0 0" rpy="0 0 0"/>
+                <geometry>
+                    <mesh filename="package://iiwa_14_r820_robot_description/meshes/link3.dae" scale="1 1 1"/>
                 </geometry>
             </collision>
@@ -111,11 +111,11 @@
                 <origin xyz="0 0 0" rpy="0 0 0"/>
                 <geometry>
-                    <mesh filename="package://iiwa_14_r850_robot_description/meshes/link4.dae" scale="1 1 1"/>
-                </geometry>
-            </visual>
-            <collision>
-                <origin xyz="0 0 0" rpy="0 0 0"/>
-                <geometry>
-                    <mesh filename="package://iiwa_14_r850_robot_description/meshes/link4.dae" scale="1 1 1"/>
+                    <mesh filename="package://iiwa_14_r820_robot_description/meshes/link4.dae" scale="1 1 1"/>
+                </geometry>
+            </visual>
+            <collision>
+                <origin xyz="0 0 0" rpy="0 0 0"/>
+                <geometry>
+                    <mesh filename="package://iiwa_14_r820_robot_description/meshes/link4.dae" scale="1 1 1"/>
                 </geometry>
             </collision>
@@ -138,11 +138,11 @@
                 <origin xyz="0 0 0" rpy="0 0 0"/>
                 <geometry>
-                    <mesh filename="package://iiwa_14_r850_robot_description/meshes/link5.dae" scale="1 1 1"/>
-                </geometry>
-            </visual>
-            <collision>
-                <origin xyz="0 0 0" rpy="0 0 0"/>
-                <geometry>
-                    <mesh filename="package://iiwa_14_r850_robot_description/meshes/link5.dae" scale="1 1 1"/>
+                    <mesh filename="package://iiwa_14_r820_robot_description/meshes/link5.dae" scale="1 1 1"/>
+                </geometry>
+            </visual>
+            <collision>
+                <origin xyz="0 0 0" rpy="0 0 0"/>
+                <geometry>
+                    <mesh filename="package://iiwa_14_r820_robot_description/meshes/link5.dae" scale="1 1 1"/>
                 </geometry>
             </collision>
@@ -165,11 +165,11 @@
                 <origin xyz="0 0 0" rpy="0 0 0"/>
                 <geometry>
-                    <mesh filename="package://iiwa_14_r850_robot_description/meshes/link6.dae" scale="1 1 1"/>
-                </geometry>
-            </visual>
-            <collision>
-                <origin xyz="0 0 0" rpy="0 0 0"/>
-                <geometry>
-                    <mesh filename="package://iiwa_14_r850_robot_description/meshes/link6.dae" scale="1 1 1"/>
+                    <mesh filename="package://iiwa_14_r820_robot_description/meshes/link6.dae" scale="1 1 1"/>
+                </geometry>
+            </visual>
+            <collision>
+                <origin xyz="0 0 0" rpy="0 0 0"/>
+                <geometry>
+                    <mesh filename="package://iiwa_14_r820_robot_description/meshes/link6.dae" scale="1 1 1"/>
                 </geometry>
             </collision>
@@ -192,11 +192,11 @@
                 <origin xyz="0 0 0" rpy="0 0 0"/>
                 <geometry>
-                    <mesh filename="package://iiwa_14_r850_robot_description/meshes/link7.dae" scale="1 1 1"/>
-                </geometry>
-            </visual>
-            <collision>
-                <origin xyz="0 0 0" rpy="0 0 0"/>
-                <geometry>
-                    <mesh filename="package://iiwa_14_r850_robot_description/meshes/link7.dae" scale="1 1 1"/>
+                    <mesh filename="package://iiwa_14_r820_robot_description/meshes/link7.dae" scale="1 1 1"/>
+                </geometry>
+            </visual>
+            <collision>
+                <origin xyz="0 0 0" rpy="0 0 0"/>
+                <geometry>
+                    <mesh filename="package://iiwa_14_r820_robot_description/meshes/link7.dae" scale="1 1 1"/>
                 </geometry>
             </collision>
