Commit message: add camera on link6

File: iiwa_14_r820_robot_description/urdf/gazebo.urdf.xacro (robot description, xacro)
@@ -7,3 +7,42 @@
         </plugin>
     </gazebo>
+    <gazebo reference="camera_link">
+        <sensor type="camera" name="camera">
+        <update_rate>30.0</update_rate>
+        <camera name="tip_link_camera">
+            <horizontal_fov>1.3962634</horizontal_fov>
+            <image>
+                <width>800</width>
+                <height>800</height>
+                <format>R8G8B8</format>
+            </image>
+            <clip>
+                <near>0.02</near>
+                <far>300</far>
+            </clip>
+            <noise>
+                <type>gaussian</type>
+                <!-- Noise is sampled independently per pixel on each frame.
+                    That pixel's noise value is added to each of its color
+                    channels, which at that point lie in the range [0,1]. -->
+                <mean>0.0</mean>
+                <stddev>0.007</stddev>
+            </noise>
+        </camera>
+            <plugin name="camera_controller" filename="libgazebo_ros_camera.so">
+            <alwaysOn>true</alwaysOn>
+            <updateRate>0.0</updateRate>
+            <cameraName>camera</cameraName>
+            <imageTopicName>image_raw</imageTopicName>
+            <cameraInfoTopicName>camera_info</cameraInfoTopicName>
+            <frameName>camera_link</frameName>
+            <hackBaseline>0.07</hackBaseline>
+            <distortionK1>0.0</distortionK1>
+            <distortionK2>0.0</distortionK2>
+            <distortionK3>0.0</distortionK3>
+            <distortionT1>0.0</distortionT1>
+            <distortionT2>0.0</distortionT2>
+            </plugin>
+        </sensor>
+    </gazebo>
 </robot>

File: iiwa_14_r820_robot_description/urdf/robot.urdf.xacro (robot description, xacro)
@@ -8,3 +8,27 @@
         <origin xyz="0 0 0" rpy="0 0 0"/>
     </xacro:iiwa_14_r820>
+    <link name="camera_link">
+        <visual>
+            <origin xyz="0 0 0" rpy="0 0 0"/>
+            <geometry>
+                <box size="0.05 0.05 0.05"/>
+            </geometry>
+        </visual>
+        <collision>
+            <origin xyz="0 0 0" rpy="0 0 0"/>
+            <geometry>
+                <box size="0.1 0.1 0.1"/>
+            </geometry>
+        </collision>
+        <inertial>
+            <mass value="0.01"/>
+            <origin xyz="0 0 0" rpy="0 0 0"/>
+            <inertia ixx="0.0001" ixy="0.0" ixz="0.0" iyy="0.0001" iyz="0.0" izz="0.0001"/>
+        </inertial>
+    </link>
+    <joint name="camera_fixed_joint" type="fixed">
+        <parent link="link6"/>
+        <child link="camera_link"/>
+        <origin xyz="0.09 0 0.05" rpy="0 ${-pi/2} 0"/>
+    </joint>
 </robot>
